File: evalboard2/evalboard2.kicad_pcb (KiCad board)
At the start: 2 copper layers, 31 parts, among them J1 USB_OTG, J11 Conn_01x18_Male, J2 power in, J9 Conn_01x17_Male, SW1 SW_Push, U1 GA144A12, U2 FT234XD-R, U3 LTC3406ES5-1.8, U4 SST25WF080B, U5 CY62167EV18, Y1 Crystal

Commit message: update
Parts:
- moved J9 75.4 mm to (194.1, 100.8), turned to 180 degrees
- moved U5 74.4 mm to (213.6, 89.2), turned to 180 degrees
- moved U4 74.1 mm to (201.1, 88.8)
- moved U1 49.3 mm to (213.9, 75.2)
- moved C5 39.4 mm to (199.7, 78.2)
- moved U2 35.8 mm to (202.9, 48.0)
- moved C3 33.9 mm to (205.2, 71.9)
- moved C11 32.7 mm to (212.1, 43.9)
- moved J1 31.5 mm to (213.4, 60.2), turned to 180 degrees
- moved C4 29.0 mm to (228.6, 78.0)
- moved J11 28.4 mm to (232.4, 54.9)
- moved C6 27.6 mm to (207.8, 68.1)
- moved C7 26.9 mm to (226.8, 71.9)
Routing:
- net a0: track 0.00 -> 36.7 mm
- net a1: track 0.00 -> 33.7 mm
- net a3: track 0.00 -> 27.6 mm
- net d13: track 0.00 -> 27.0 mm, vias 0 -> 2
- net d0: track 0.00 -> 25.0 mm
- net d1: track 0.00 -> 24.9 mm
- net a2: track 0.00 -> 24.7 mm
- net d14: track 0.00 -> 23.6 mm, vias 0 -> 2
- net a5: track 0.00 -> 23.6 mm
- net d2: track 0.00 -> 23.0 mm
- net d3: track 0.00 -> 22.2 mm
- net d4: track 0.00 -> 20.4 mm
- net d15: track 0.00 -> 19.2 mm, vias 0 -> 2
- net d5: track 0.00 -> 18.9 mm
- net 008.17: track 0.00 -> 17.8 mm, vias 0 -> 2
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Other:
- net class Default: clearance 0.2 -> 0.127; trace_width 0.25 -> 0.127
- rule trace_clearance: 0.2 -> 0.127
- rule trace_min: 0.16 -> 0.127
