File: evalboard2/evalboard2.sch (KiCad schematic (older format))
At the start: 31 parts, among them J1 USB_OTG, J11 Conn_01x18_Male, J2 power in, J9 Conn_01x17_Male, SW1 SW_Push, U1 GA144A12, U2 FT234XD-R, U3 LTC3406ES5-1.8, U4 SST25WF080B, U5 CY62167EV18, Y1 Crystal

Commit message: update
Parts:
- removed J9: Conn_01x17_Male, Connector_PinHeader_2.54mm:PinHeader_1x17_P2.54mm_Vertical, symbol Connector:Conn_01x17_Male
- added J3: Conn_01x18_Male, Connector_PinHeader_2.54mm:PinHeader_1x18_P2.54mm_Vertical, symbol Connector:Conn_01x18_Male
Connections:
- net 500.17: now also J3.1 (Pin_1)
- net 600.17: now also J3.2 (Pin_2)
- net 701.1: now also J3.3 (Pin_3)
- net 701.17: now also J3.4 (Pin_4)
- net 705.1: now also J3.8 (Pin_8)
- net 705.17: now also J3.5 (Pin_5)
- net 705.3: now also J3.7 (Pin_7)
- net 705.5: now also J3.6 (Pin_6)
- net 708.1: now also J3.9 (Pin_9)
- net 708.17: now also J3.10 (Pin_10)
- net 709.ai: now also J3.12 (Pin_12)
- net 709.ao: now also J3.11 (Pin_11)
- net 713.ao: now also J3.14 (Pin_14)
- net 713ai: now also J3.13 (Pin_13)
- net 715.17: now also J3.15 (Pin_15)
- net 717.ai: now also J3.17 (Pin_17)
- net 717.ao: now also J3.16 (Pin_16)
- net GND: now also J3.18 (Pin_18)
Changed lines of the file:
@@
 EESchema Schematic File Version 4
+LIBS:evalboard2-cache
 EELAYER 26 0
 EELAYER END
@@
 715.17
 $Comp
-L Connector:Conn_01x17_Male J9
-U 1 1 5CB7C03A
-P 9550 5450
-F 0 "J9" H 9656 6428 50  0000 C CNN
-F 1 "Conn_01x17_Male" H 9656 6337 50  0000 C CNN
-F 2 "Connector_PinHeader_2.54mm:PinHeader_1x17_P2.54mm_Vertical" H 9550 5450 50  0001 C CNN
-F 3 "~" H 9550 5450 50  0001 C CNN
-	1    9550 5450
-	1    0    0    -1
-$EndComp
-$Comp
 L Connector:Conn_01x18_Male J11
 U 1 1 5CBB90C5
@@
 P 6900 4400
 F 0 "U5" H 7025 5378 50  0000 C CNN
-F 1 "CY62167EV18" H 7025 5287 50  0000 C CNN
+F 1 "CY62167EV18" H 6950 4150 50  0000 C CNN
 F 2 "ga144:CY62167EV18LL" H 7450 5100 50  0001 C CNN
 F 3 "" H 7450 5100 50  0001 C CNN
@@
 $EndComp
 Connection ~ 2800 7300
+$Comp
+L Connector:Conn_01x18_Male J3
+U 1 1 5C0DF0F3
+P 9550 5450
+F 0 "J3" H 9656 6428 50  0000 C CNN
+F 1 "Conn_01x18_Male" H 9656 6337 50  0000 C CNN
+F 2 "Connector_PinHeader_2.54mm:PinHeader_1x18_P2.54mm_Vertical" H 9550 5450 50  0001 C CNN
+F 3 "~" H 9550 5450 50  0001 C CNN
+	1    9550 5450
+	1    0    0    -1
+$EndComp
+$Comp
+L power:GND #PWR0108
+U 1 1 5C0DF289
+P 9750 6350
+F 0 "#PWR0108" H 9750 6100 50  0001 C CNN
+F 1 "GND" V 9755 6222 50  0000 R CNN
+F 2 "" H 9750 6350 50  0001 C CNN
+F 3 "" H 9750 6350 50  0001 C CNN
+	1    9750 6350
+	0    -1   -1   0
+$EndComp
 $EndSCHEMATC
