File: breakout/breakout.kicad_pcb (KiCad board)
At the start: 2 copper layers, 52.3 x 52.5 mm, 10 parts, among them J1 Conn_01x20_Male, J5 Conn_01x18_Male, J7 Conn_01x18_Male, J8 Conn_01x18_Male, U1 GA144A12

Commit message: breakout changes
Other:
- board text added: "GA144 breakout version 1 github.com/mschuldt/ga144-breakout"
Changed lines of the file:
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@@
-(kicad_pcb (version 20171130) (host pcbnew 5.0.1-33cea8e~68~ubuntu14.04.1)
+(kicad_pcb (version 20171130) (host pcbnew 5.0.2-bee76a0~70~ubuntu14.04.1)
   (general
     (thickness 1.6)
-    (drawings 152)
+    (drawings 153)
     (tracks 289)
     (zones 0)
@@
   )
   (setup
-    (last_trace_width 0.16)
+    (last_trace_width 0.25)
     (user_trace_width 0.16)
     (user_trace_width 0.2)
@@
     )
   )
+  (gr_text "GA144 breakout version 1\ngithub.com/mschuldt/ga144-breakout" (at 151.638 109.982) (layer B.SilkS)
+    (effects (font (size 1.5 1.5) (thickness 0.3)) (justify left mirror))
+  )
   (gr_line (start 105.156 66.294) (end 108.966 70.612) (layer F.SilkS) (width 0.2))
