File: breakout/breakout.sch (KiCad schematic (older format))
At the start: 10 parts, among them J1 Conn_01x20_Male, J5 Conn_01x18_Male, J7 Conn_01x18_Male, J8 Conn_01x18_Male, U1 GA144A12

Commit message: breakout changes
Parts:
- U1: symbol ak-ga144:GA144A12 -> breakout-rescue:GA144A12-ak-ga144
Changed lines of the file:
@@
 $EndDescr
 $Comp
-L ak-ga144:GA144A12 U1
+L breakout-rescue:GA144A12-ak-ga144 U1
 U 1 1 5BE088A7
 P 3000 3300
